File: pcb/stm32f4_remote_controller.kicad_pcb (KiCad board)
At the start: 2 copper layers, 0 parts

Commit message: pcb: add first version of pcb
Parts:
- added BT1: 3V, Battery:BatteryHolder_Keystone_2468_2xAAA, B.Cu at (191.3, 62.6)
- added C1: 100n, Capacitor_SMD:C_0402_1005Metric, F.Cu at (88.0, 54.8)
- added C10: 1u, Capacitor_SMD:C_0603_1608Metric, F.Cu at (159.0, 54.6)
- added C11: 10u, Capacitor_SMD:C_0603_1608Metric, F.Cu at (169.0, 45.0)
- added C12: 10p, Capacitor_SMD:C_0201_0603Metric, F.Cu at (164.3, 60.5)
- added C13: 22u, Capacitor_SMD:C_0805_2012Metric, F.Cu at (142.4, 52.8)
- added C14: 22u, Capacitor_SMD:C_0805_2012Metric, F.Cu at (142.4, 56.2)
- added C15: 2,2u, Capacitor_SMD:C_0603_1608Metric, F.Cu at (159.0, 59.6)
- added C2: 100n, Capacitor_SMD:C_0402_1005Metric, F.Cu at (84.8, 54.8)
- added C3: 100n, Capacitor_SMD:C_0402_1005Metric, F.Cu at (172.3, 50.2)
- added C4: 100n, Capacitor_SMD:C_0402_1005Metric, F.Cu at (81.7, 54.8)
- added C5: 100n, Capacitor_SMD:C_0402_1005Metric, F.Cu at (78.5, 54.8)
- added C6: 10u, Capacitor_SMD:C_0603_1608Metric, F.Cu at (74.7, 54.8)
- added C7: 100n, Capacitor_SMD:C_0402_1005Metric, F.Cu at (163.1, 49.4)
- added C8: 20p, Capacitor_SMD:C_0201_0603Metric, F.Cu at (78.4, 61.9)
- added C9: 20p, Capacitor_SMD:C_0201_0603Metric, F.Cu at (78.4, 58.9)
- added FB1: FerriteBead, Inductor_SMD:L_0603_1608Metric, F.Cu at (159.0, 62.1)
- added J1: Conn_01x04_Pin, Connector_PinHeader_2.54mm:PinHeader_1x04_P2.54mm_Vertical, F.Cu at (115.0, 51.0)
- added L1: 0.47u, Inductor_SMD:L_01005_0402Metric, F.Cu at (164.2, 62.2)
- added R1: 10k, Resistor_SMD:R_0402_1005Metric, F.Cu at (162.4, 51.8)
- added R2: 10K, Resistor_SMD:R_0402_1005Metric, F.Cu at (162.4, 53.8)
- added R3: 10K, Resistor_SMD:R_0402_1005Metric, F.Cu at (162.4, 55.8)
- added R4: 316K, Resistor_SMD:R_0805_2012Metric, F.Cu at (169.8, 56.5)
- added R5: 100K, Resistor_SMD:R_0805_2012Metric, F.Cu at (169.8, 59.4)
- added R6: 1K, Resistor_SMD:R_0402_1005Metric, F.Cu at (159.1, 67.2)
- added R7: 1K, Resistor_SMD:R_0402_1005Metric, F.Cu at (176.9, 49.2)
- added R8: 10K, Resistor_SMD:R_0402_1005Metric, F.Cu at (162.4, 61.8)
- added R9: 1K, Resistor_SMD:R_0402_1005Metric, F.Cu at (162.4, 63.8)
- added SW1: DISPLAY_BUTTON, Button_Switch_THT:Push_E-Switch_KS01Q01, F.Cu at (115.6, 98.0)
- added SW2: SW_DPDT_x2, Button_Switch_THT:SW_CK_JS202011AQN_DPDT_Angled, F.Cu at (169.2, 63.9)
- added SW3: RESET_BUTTON, Button_Switch_THT:SW_PUSH-12mm, F.Cu at (56.5, 69.8)
- added U1: STM32F401CCU6, Package_DFN_QFN:QFN-48-1EP_7x7mm_P0.5mm_EP5.6x5.6mm, F.Cu at (85.2, 60.8)
- added U2: OLED DISPLAY, OLED-DISPLAY-128x64:MODULE_DM-OLED096-636, F.Cu at (118.6, 76.0)
- added U3: ~, Connector_Molex:Molex_SL_171971-0006_1x06_P2.54mm_Vertical, F.Cu at (45.8, 103.0)
- added U4: ~, Connector_Molex:Molex_SL_171971-0005_1x05_P2.54mm_Vertical, F.Cu at (79.8, 107.0)
- added U5: ~, Connector_Molex:Molex_SL_171971-0005_1x05_P2.54mm_Vertical, F.Cu at (147.0, 107.2)
- added U6: TPS61021ADSGR, dc-dc_step-up:SON50P200X200X80-9N, F.Cu at (164.8, 45.8)
- added Y1: 8Mhz, Crystal:Crystal_SMD_5032-4Pin_5.0x3.2mm, F.Cu at (75.4, 60.2)
