File: pcb/stm32f4_remote_controller.kicad_pcb (KiCad board)
At the start: 2 copper layers, 38 parts, among them J1 Conn_01x04_Pin, SW1 DISPLAY_BUTTON, SW2 SW_DPDT_x2, SW3 RESET_BUTTON, U1 STM32F401CCU6, U2 OLED DISPLAY, U6 TPS61021ADSGR, Y1 8Mhz

Commit message: pcb: add ready pcb
Parts:
- added G***: LOGO, logo:cf_embedded, F.Cu at (121.0, 115.5)
- added H1: MountingHole, MountingHole:MountingHole_2.5mm, F.Cu at (102.5, 61.0)
- added H2: MountingHole, MountingHole:MountingHole_2.5mm, F.Cu at (102.5, 123.0)
- added H3: MountingHole, MountingHole:MountingHole_2.5mm, F.Cu at (159.0, 61.0)
- added H4: MountingHole, MountingHole:MountingHole_2.5mm, F.Cu at (159.0, 123.0)
- BT1: footprint Battery:BatteryHolder_Keystone_2468_2xAAA -> Connector_Phoenix_GMSTB:PhoenixContact_GMSTBA_2,5_2-G-7,62_1x02_P7.62mm_Horizontal; moved to F.Cu
- C12, C8, C9: footprint Capacitor_SMD:C_0201_0603Metric -> Capacitor_SMD:C_0402_1005Metric
- FB1: value FerriteBead -> 120R
- L1: footprint Inductor_SMD:L_01005_0402Metric -> Inductor_SMD:L_1206_3216Metric
- SW1: footprint Button_Switch_THT:Push_E-Switch_KS01Q01 -> Connector_PinHeader_2.54mm:PinHeader_1x02_P2.54mm_Vertical
- SW3: footprint Button_Switch_THT:SW_PUSH-12mm -> Button_Switch_THT:SW_PUSH_6mm
- U2: footprint OLED-DISPLAY-128x64:MODULE_DM-OLED096-636 -> Connector_PinHeader_2.54mm:PinHeader_1x04_P2.54mm_Vertical
- U4, U5: footprint Connector_Molex:Molex_SL_171971-0005_1x05_P2.54mm_Vertical -> Connector_PinHeader_2.54mm:PinHeader_1x05_P2.54mm_Vertical
- moved R7 81.2 mm to (134.8, 118.6), turned to 90 degrees
- moved C11 79.1 mm to (139.7, 118.5)
- moved R1 77.7 mm to (111.5, 110.5), turned to 90 degrees
- moved U6 73.4 mm to (135.4, 113.0), turned to -90 degrees
- moved SW2 68.9 mm to (132.5, 122.2)
- moved C5 68.5 mm to (129.0, 101.0), turned to 180 degrees
- moved BT1 68.0 mm to (147.7, 114.8), turned to 90 degrees
- moved Y1 67.4 mm to (140.5, 77.5), turned to 180 degrees
- moved C9 65.5 mm to (140.0, 81.0), turned to 0 degrees
- moved C4 64.8 mm to (129.0, 99.0), turned to 180 degrees
- moved C6 64.7 mm to (129.0, 90.0), turned to 180 degrees
- moved R4 64.2 mm to (133.1, 109.2)
- moved J1 63.9 mm to (159.0, 97.3), turned to 180 degrees
- moved SW3 63.8 mm to (120.2, 67.8)
- moved C3 63.8 mm to (129.0, 97.0), turned to 180 degrees
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Connections:
- C12 pad 1: /STEP_UP_3.3V -> +STEP_UP_3.3V
- C13 pad 1: /STEP_UP_3.3V -> +STEP_UP_3.3V
- C14 pad 1: /STEP_UP_3.3V -> +STEP_UP_3.3V
- R4 pad 1: /STEP_UP_3.3V -> +STEP_UP_3.3V
- R6 pad 2: ADC1_IN0_BATT_VOLTAGE -> ADC1_IN4_BATT_VOLTAGE
- U1 pad 10: ADC1_IN0_BATT_VOLTAGE -> ADC1_IN0_SPEED_CONTROL
- U1 pad 11: ADC1_IN1_SPEED_CONTROL -> ADC1_IN1_ANGLE_CONTROL
- U1 pad 12: ADC1_IN2_ANGLE_CONTROL -> USART2_TX
- U1 pad 13: unconnected-(U1-PA3-Pad13) -> USART2_RX
- U1 pad 14: DISPLAY_BUTTON_INPUT -> ADC1_IN4_BATT_VOLTAGE
- U1 pad 15: HM_10_STATE -> unconnected-(U1-PA5-Pad15)
- U1 pad 30: USART1_TX -> unconnected-(U1-PA9-Pad30)
- U1 pad 31: USART1_RX -> unconnected-(U1-PA10-Pad31)
- U1 pad 41: unconnected-(U1-PB5-Pad41) -> DISPLAY_BUTTON_INPUT
- U3 pad 2: HM_10_STATE -> GND
- U3 pad 3: USART1_TX -> USART2_TX
- U3 pad 4: USART1_RX -> USART2_RX
- U4 pad 2: ADC1_IN1_SPEED_CONTROL -> ADC1_IN0_SPEED_CONTROL
- U5 pad 3: ADC1_IN2_ANGLE_CONTROL -> ADC1_IN1_ANGLE_CONTROL
- U6 pad 3: /STEP_UP_3.3V -> +STEP_UP_3.3V
- U6 pad 4: /STEP_UP_3.3V -> +STEP_UP_3.3V
Routing:
- net +STEP_UP_3.3V: track 0.00 -> 197.9 mm, vias 0 -> 4
- net GND: track 0.00 -> 52.7 mm, vias 0 -> 28
- net USART2_RX: track 0.00 -> 35.7 mm
- net USART2_TX: track 0.00 -> 35.6 mm
- net ADC1_IN0_SPEED_CONTROL: track 0.00 -> 34.2 mm
- net ADC1_IN1_ANGLE_CONTROL: track 0.00 -> 32.3 mm
- net I2C1_SDA: track 0.00 -> 29.5 mm
- net RESET_PIN: track 0.00 -> 28.7 mm
- net I2C1_SCL: track 0.00 -> 27.9 mm
- net /SWDIO: track 0.00 -> 24.2 mm
- net /SWCLK: track 0.00 -> 21.3 mm
- net Net-(U6-AGND): track 0.00 -> 21.2 mm
- net Net-(BT1-+): track 0.00 -> 19.7 mm
- net DISPLAY_BUTTON_INPUT: track 0.00 -> 16.6 mm
- net Net-(C7-Pad1): track 0.00 -> 13.3 mm
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- added copper zone on B.Cu, net GND
Other:
- board text added: "ANGLE CONTROL"
- board text added: "HM-10"
- board text added: "OLED-DISPLAY"
- board text added: "SPEED CONTROL"
- board text added: "SWD"
